File: Schemat_eagle/esc_ne5551.brd (EAGLE design)
At the start: 31.7 x 32.1 mm, 11 parts, among them IC1 NE555, IC2 TL071P, Q1 IRF510

Commit message: Add files via upload
Parts:
- moved IC2 2.11 mm to (28.7, 28.2)
- moved R1 2.11 mm to (29.6, 40.5)
- moved Q1 2.11 mm to (14.2, 21.8)
- moved R4 2.11 mm to (16.1, 29.2)
- moved X1 2.11 mm to (9.40, 43.1)
- moved X2 2.11 mm to (9.40, 32.9)
- moved C1 2.11 mm to (16.4, 36.1)
- moved IC1 2.11 mm to (19.9, 43.3)
- moved R2 2.11 mm to (26.9, 40.5)
- moved R3 2.11 mm to (29.3, 20.7)
- moved C2 2.11 mm to (16.3, 32.8)
Routing:
- net +12V: track 66.9 -> 70.1 mm
Other:
- board size 31.7 x 32.1 mm -> 36.9 x 36.7 mm
- board text added: "MARCIN PRZĄDKA 219793"
- board text removed: "219793"
